File: GPS-DO_BreakoutBoard/GPS-DO_BreakoutBoard.kicad_sch (KiCad schematic)
At the start: 23 parts, among them J1 Conn_Coaxial, J2 Conn_Coaxial, J3 Conn_Coaxial, J4 FTDI Cable, J5 Conn_01x02_Socket

Commit message: added 3d view and schematic pdf
Other:
- company: (none) -> NCSU - AERPAW
- title: (none) -> GPS-DO Breakout Board
Changed lines of the file:
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@@
 (kicad_sch (version 20230121) (generator eeschema)
   (paper "A4")
+  (title_block
+    (title "GPS-DO Breakout Board")
+    (date "2023-06-09")
+    (rev "V0.1")
+    (company "NCSU - AERPAW")
+    (comment 1 "Author: Mark Funderburk")
+  )
   (junction (at 158.75 113.03) (diameter 0) (color 0 0 0 0)
   )

Commit message: V1.0 Submitted for ordering
Parts:
- added C3: 47uF, Capacitor_SMD:C_1206_3216Metric, symbol Device:C_Small
- added D10: LED, LED_SMD:LED_1206_3216Metric, symbol Device:LED
- added R3: 1k, Resistor_SMD:R_1206_3216Metric, symbol Device:R_Small_US
Connections:
- net GND: now also C3.2, D10.1 (K)
- net at U1.3 (Lock_OK): now also R3.1
- net at U1.6 (5V_OUT): now also C3.1
- new net: D10.2 (A), R3.2
- no-connect marks 7 -> 5
Changed lines of the file:
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@@
   (junction (at 129.54 48.26) (diameter 0) (color 0 0 0 0)
   )
+  (junction (at 132.08 113.03) (diameter 0) (color 0 0 0 0)
+  )
   (junction (at 255.27 29.21) (diameter 0) (color 0 0 0 0)
   )
@@
   (junction (at 146.05 29.21) (diameter 0) (color 0 0 0 0)
   )
+  (junction (at 139.7 113.03) (diameter 0) (color 0 0 0 0)
+  )
   (junction (at 213.36 29.21) (diameter 0) (color 0 0 0 0)
   )
@@
   (junction (at 59.69 69.85) (diameter 0) (color 0 0 0 0)
   )
-  (no_connect (at 144.78 90.17))
   (no_connect (at 34.29 74.93))
   (no_connect (at 34.29 64.77))
   (no_connect (at 173.99 99.06))
-  (no_connect (at 144.78 97.79))
   (no_connect (at 173.99 91.44))
   (no_connect (at 173.99 93.98))
@@
     (stroke (width 0) (type default))
   )
+  (wire (pts (xy 116.84 110.49) (xy 116.84 113.03))
+    (stroke (width 0) (type default))
+  )
   (wire (pts (xy 107.95 48.26) (xy 90.17 48.26))
     (stroke (width 0) (type default))
@@
     (stroke (width 0) (type default))
   )
+  (wire (pts (xy 132.08 110.49) (xy 132.08 113.03))
+    (stroke (width 0) (type default))
+  )
   (wire (pts (xy 34.29 29.21) (xy 63.5 29.21))
     (stroke (width 0) (type default))
@@
     (stroke (width 0) (type default))
   )
+  (wire (pts (xy 116.84 113.03) (xy 132.08 113.03))
+    (stroke (width 0) (type default))
+  )
   (wire (pts (xy 139.7 100.33) (xy 139.7 85.09))
     (stroke (width 0) (type default))
@@
     (stroke (width 0) (type default))
   )
+  (wire (pts (xy 116.84 100.33) (xy 116.84 102.87))
+    (stroke (width 0) (type default))
+  )
   (wire (pts (xy 34.29 69.85) (xy 59.69 69.85))
     (stroke (width 0) (type default))
@@
     (stroke (width 0) (type default))
   )
+  (wire (pts (xy 116.84 90.17) (xy 116.84 95.25))
+    (stroke (width 0) (type default))
+  )
   (wire (pts (xy 53.34 19.05) (xy 63.5 19.05))
     (stroke (width 0) (type default))
@@
     (stroke (width 0) (type default))
   )
+  (wire (pts (xy 144.78 97.79) (xy 132.08 97.79))
+    (stroke (width 0) (type default))
+  )
   (wire (pts (xy 146.05 29.21) (xy 146.05 31.75))
     (stroke (width 0) (type default))
@@
     (stroke (width 0) (type default))
   )
+  (wire (pts (xy 132.08 97.79) (xy 132.08 105.41))
+    (stroke (width 0) (type default))
+  )
   (wire (pts (xy 213.36 29.21) (xy 213.36 71.12))
     (stroke (width 0) (type default))
@@
     (stroke (width 0) (type default))
   )
+  (wire (pts (xy 144.78 90.17) (xy 116.84 90.17))
+    (stroke (width 0) (type default))
+  )
   (wire (pts (xy 232.41 140.97) (xy 232.41 144.78))
     (stroke (width 0) (type default))
   )
   (wire (pts (xy 246.38 78.74) (xy 246.38 85.09))
+    (stroke (width 0) (type default))
+  )
+  (wire (pts (xy 132.08 113.03) (xy 139.7 113.03))
     (stroke (width 0) (type default))
   )
@@
         (path "/79d0db63-5189-42f4-b66e-58a4c192f9d9"
           (reference "D4") (unit 1)
+        )
+      )
+    )
+  )
+  (symbol (lib_id "Device:R_Small_US") (at 116.84 97.79 0) (unit 1)
+    (in_bom yes) (on_board yes) (dnp no)
+    (property "Reference" "R3" (at 118.11 96.52 0)
+      (effects (font (size 1.27 1.27)) (justify left))
+    )
+    (property "Value" "1k" (at 118.11 99.314 0)
+      (effects (font (size 1.27 1.27)) (justify left))
+    )
+    (property "Footprint" "Resistor_SMD:R_1206_3216Metric" (at 116.84 97.79 0)
+      (effects (font (size 1.27 1.27)) hide)
+    )
+    (property "Datasheet" "~" (at 116.84 97.79 0)
+      (effects (font (size 1.27 1.27)) hide)
+    )
+    (pin "1")
+    (pin "2")
+    (instances
+      (project "GPS-DO_BreakoutBoard"
+        (path "/79d0db63-5189-42f4-b66e-58a4c192f9d9"
+          (reference "R3") (unit 1)
+        )
+      )
+    )
+  )
+  (symbol (lib_id "Device:LED") (at 116.84 106.68 90) (unit 1)
+    (in_bom yes) (on_board yes) (dnp no)
+    (property "Reference" "D10" (at 114.3 106.68 0)
+      (effects (font (size 1.27 1.27)))
+    )
+    (property "Value" "LED" (at 119.38 106.68 0)
+      (effects (font (size 1.27 1.27)))
+    )
+    (property "Footprint" "LED_SMD:LED_1206_3216Metric" (at 116.84 106.68 0)
+      (effects (font (size 1.27 1.27)) hide)
+    )
+    (property "Datasheet" "~" (at 116.84 106.68 0)
+      (effects (font (size 1.27 1.27)) hide)
+    )
+    (pin "1")
+    (pin "2")
+    (instances
+      (project "GPS-DO_BreakoutBoard"
+        (path "/79d0db63-5189-42f4-b66e-58a4c192f9d9"
+          (reference "D10") (unit 1)
         )
       )
@@
         )
       )
+    )
+  )
+  (symbol (lib_id "Device:C_Small") (at 132.08 107.95 0) (unit 1)
+    (in_bom yes) (on_board yes) (dnp no)
+    (property "Reference" "C3" (at 132.334 106.172 0)
+      (effects (font (size 1.27 1.27)) (justify left))
+    )
+    (property "Value" "47uF" (at 132.334 109.982 0)
+      (effects (font (size 1.27 1.27)) (justify left))
+    )
+    (property "Footprint" "Capacitor_SMD:C_1206_3216Metric" (at 132.08 107.95 0)
+      (effects (font (size 1.27 1.27)) hide)
+    )
+    (property "Datasheet" "~" (at 132.08 107.95 0)
+      (effects (font (size 1.27 1.27)) hide)
+    )
+    (pin "1")
+    (pin "2")
+    (instances
+      (project "GPS-DO_BreakoutBoard"
+        (path "/79d0db63-5189-42f4-b66e-58a4c192f9d9"
+          (reference "C3") (unit 1)
+        )
+      )
